Commit message: paper ready. experiments completed

File: kfp_v2/digit/models/buff_digit/prost_digit_hover.urdf (robot description, URDF)
Before this commit: robot buff_digit, 47 links, 46 joints
Links:
- link base_link: mass 15.028392 -> 55.028392

File: kfp_v2/digit/models/table/table.urdf (robot description, URDF)
Before this commit: robot table.urdf, 1 links, 0 joints
Links:
- added link guard, mass .0; collision box size=1.5 0.025 0.125; visual box size=1.5 0.025 0.125
- added link left_guard, mass .0; collision box size=0.025 1 0.125; visual box size=0.025 1 0.125
- added link right_guard, mass .0; collision box size=0.025 1 0.125; visual box size=0.025 1 0.125
Joints:
- added joint guard_to_surface: type fixed, parent baseLink, child guard, origin xyz=0 0.5 0.0625 rpy=0 0 0
- added joint left_guard_to_surface: type fixed, parent baseLink, child left_guard, origin xyz=-0.75 0 0.0625 rpy=0 0 0
- added joint right_guard_to_surface: type fixed, parent baseLink, child right_guard, origin xyz=0.75 0 0.0625 rpy=0 0 0

File: kfp_v2/digit/models/tray/tray.urdf (robot description, URDF)
Before this commit: robot tray, 1 links, 0 joints
Links:
- link baseLink: geometry collision mesh filename=tray_vhacd.obj scale=0.5 0.7 0.8; visual mesh filename=tray_vhacd.obj scale=0.5 0.7 0.8
